File: kicad/drv8304_eval/drv8304_eval.kicad_pcb (KiCad board)
At the start: 4 copper layers, 48.1 x 41.6 mm, 34 parts, among them J1 Conn_01x01_Pin, J2 Conn_01x01_Pin, J3 Conn_01x01_Pin, J6 Conn_01x01_Pin, J7 Conn_01x01_Pin, J8 Conn_01x12_Pin, Q1 CSD18514Q5A, Q2 CSD18514Q5A, Q3 CSD18514Q5A, Q4 CSD18514Q5A, Q5 CSD18514Q5A, Q6 CSD18514Q5A, U1 DRV8304HRHAR

Commit message: Fix the lack of a polarized capacitor and add INL channel to the gate driver.
Parts:
- turned C12 to 90 degrees
- turned C13 to 180 degrees
- turned C14 to -90 degrees
- turned C15 to 90 degrees
Connections:
- C12 pad 1: GND -> +BATT
- C12 pad 2: +BATT -> GND
- C13 pad 1: GND -> +BATT
- C13 pad 2: +BATT -> GND
- C14 pad 1: GND -> +BATT
- C14 pad 2: +BATT -> GND
- C15 pad 1: GND -> +BATT
- C15 pad 2: +BATT -> GND
- U1 pad 35: unconnected-(U1-INLA-Pad35) -> /INL
- U1 pad 37: unconnected-(U1-INLB-Pad37) -> /INL
- U1 pad 39: unconnected-(U1-INLC-Pad39) -> /INL
