File: kicad/drv8304_eval/drv8304_eval.kicad_sch (KiCad schematic)
At the start: 19 parts, among them J1 Conn_01x01_Pin, J2 Conn_01x01_Pin, J3 Conn_01x01_Pin, J6 Conn_01x01_Pin, J7 Conn_01x01_Pin, J8 Conn_01x12_Pin, U1 DRV8304HRHAR

Commit message: Fix the lack of a polarized capacitor and add INL channel to the gate driver.
Parts:
- C15: symbol Device:C -> Device:C_Polarized; now in the parts list
Connections:
- net +BATT: now also C15.1; no longer C15.2
- net GND: now also C15.2; no longer C15.1
- net INL: now reaches U1.35 (INLA)
- net INL: now also U1.37 (INLB), U1.39 (INLC)
- no-connect marks 3 -> 0
Changed lines of the file:
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@@
 (kicad_sch
-	(version 20260101)
+	(version 20260306)
 	(generator "eeschema")
 	(generator_version "10.0")
@@
 	)
 	(junction
+		(at 123.19 53.34)
+		(diameter 0)
+		(color 0 0 0 0)
+	)
+	(junction
+		(at 123.19 48.26)
+		(diameter 0)
+		(color 0 0 0 0)
+	)
+	(junction
 		(at 119.38 90.17)
 		(diameter 0)
@@
 		(color 0 0 0 0)
 	)
-	(no_connect
-		(at 130.81 53.34)
-	)
-	(no_connect
-		(at 130.81 58.42)
-	)
-	(no_connect
-		(at 130.81 48.26)
-	)
 	(wire
 		(pts
@@
 	(wire
 		(pts
+			(xy 123.19 48.26) (xy 123.19 53.34)
+		)
+		(stroke
+			(width 0)
+			(type default)
+		)
+	)
+	(wire
+		(pts
 			(xy 158.75 66.04) (xy 190.5 66.04)
 		)
@@
 	(wire
 		(pts
+			(xy 121.92 48.26) (xy 123.19 48.26)
+		)
+		(stroke
+			(width 0)
+			(type default)
+		)
+	)
+	(wire
+		(pts
 			(xy 119.38 87.63) (xy 119.38 90.17)
 		)
@@
 	(wire
 		(pts
+			(xy 123.19 48.26) (xy 130.81 48.26)
+		)
+		(stroke
+			(width 0)
+			(type default)
+		)
+	)
+	(wire
+		(pts
 			(xy 228.6 93.98) (xy 218.44 93.98)
 		)
@@
 	(wire
 		(pts
+			(xy 130.81 53.34) (xy 123.19 53.34)
+		)
+		(stroke
+			(width 0)
+			(type default)
+		)
+	)
+	(wire
+		(pts
+			(xy 123.19 58.42) (xy 123.19 53.34)
+		)
+		(stroke
+			(width 0)
+			(type default)
+		)
+	)
+	(wire
+		(pts
 			(xy 193.04 104.14) (xy 199.39 104.14)
 		)
@@
 	(wire
 		(pts
+			(xy 130.81 58.42) (xy 123.19 58.42)
+		)
+		(stroke
+			(width 0)
+			(type default)
+		)
+	)
+	(wire
+		(pts
 			(xy 158.75 43.18) (xy 158.75 38.1)
 		)
@@
 		)
 	)
+	(hierarchical_label "INL"
+		(shape input)
+		(at 121.92 48.26 180)
+		(effects
+			(font
+				(size 1.27 1.27)
+			)
+			(justify right)
+		)
+	)
 	(hierarchical_label "nFAULT"
 		(shape output)
@@
 	)
 	(symbol
-		(lib_id "Device:C")
-		(at 165.1 26.67 180)
+		(lib_id "Device:C_Polarized")
+		(at 165.1 26.67 0)
+		(mirror y)
 		(unit 1)
 		(body_style 1)
 		(exclude_from_sim no)
-		(in_bom no)
+		(in_bom yes)
 		(on_board yes)
 		(in_pos_files yes)
 		(dnp no)
-		(fields_autoplaced yes)
 		(property "Reference" "C15"
-			(at 168.91 25.3999 0)
+			(at 168.91 27.0511 0)
 			(show_name no)
 			(do_not_autoplace no)
@@
 		)
 		(property "Value" "150uF"
-			(at 168.91 27.9399 0)
+			(at 168.91 24.5111 0)
 			(show_name no)
 			(do_not_autoplace no)
@@
 		)
 		(property "Footprint" "Capacitor_SMD:CP_Elec_10x12.5"
-			(at 164.1348 22.86 0)
+			(at 164.1348 30.48 0)
 			(hide yes)
 			(show_name no)
@@
 			)
 		)
-		(property "Description" "Unpolarized capacitor"
+		(property "Description" "Polarized capacitor"
 			(at 165.1 26.67 0)
 			(hide yes)
@@
 		)
 		(instances
-			(project ""
+			(project "drv8304_eval"
 				(path "/74747308-ce22-44fa-9f28-8b5db5d05ff6"
 					(reference "J8")
@@
 		)
 		(instances
-			(project ""
+			(project "drv8304_eval"
 				(path "/74747308-ce22-44fa-9f28-8b5db5d05ff6"
 					(reference "D1")
@@
 		)
 		(instances
-			(project ""
+			(project "drv8304_eval"
 				(path "/74747308-ce22-44fa-9f28-8b5db5d05ff6"
 					(reference "U1")
@@
 		)
 		(instances
-			(project ""
+			(project "drv8304_eval"
 				(path "/74747308-ce22-44fa-9f28-8b5db5d05ff6"
 					(reference "R1")
@@
 		)
 		(instances
-			(project ""
+			(project "drv8304_eval"
 				(path "/74747308-ce22-44fa-9f28-8b5db5d05ff6"
 					(reference "J1")
@@
 		)
 		(instances
-			(project ""
+			(project "drv8304_eval"
 				(path "/74747308-ce22-44fa-9f28-8b5db5d05ff6"
 					(page "2")
