File: kicad/drv8304_eval/half_bridge.kicad_sch (KiCad schematic)
At the start: 5 parts, among them Q1 CSD18514Q5A, Q2 CSD18514Q5A

Commit message: Fix the lack of a polarized capacitor and add INL channel to the gate driver.
Parts:
- C12: symbol Device:C -> Device:C_Polarized; now in the parts list
Connections:
- net +BATT: now also C12.1; no longer C12.2
- net GND: now also C12.2; no longer C12.1
Changed lines of the file:
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@@
 (kicad_sch
-	(version 20260101)
+	(version 20260306)
 	(generator "eeschema")
 	(generator_version "10.0")
@@
 	)
 	(symbol
-		(lib_id "Device:C")
-		(at 153.67 55.88 180)
+		(lib_id "Device:C_Polarized")
+		(at 153.67 55.88 0)
+		(mirror y)
 		(unit 1)
 		(body_style 1)
 		(exclude_from_sim no)
-		(in_bom no)
+		(in_bom yes)
 		(on_board yes)
 		(in_pos_files yes)
 		(dnp no)
-		(fields_autoplaced yes)
 		(property "Reference" "C12"
-			(at 157.48 54.6099 0)
+			(at 157.48 56.2611 0)
 			(show_name no)
 			(do_not_autoplace no)
@@
 		)
 		(property "Value" "150uF"
-			(at 157.48 57.1499 0)
+			(at 157.48 53.7211 0)
 			(show_name no)
 			(do_not_autoplace no)
@@
 		)
 		(property "Footprint" "Capacitor_SMD:CP_Elec_10x12.5"
-			(at 152.7048 52.07 0)
+			(at 152.7048 59.69 0)
 			(hide yes)
 			(show_name no)
@@
 			)
 		)
-		(property "Description" "Unpolarized capacitor"
+		(property "Description" "Polarized capacitor"
 			(at 153.67 55.88 0)
 			(hide yes)
