File: kicad/stm32_g4_main_board/board/_restore_backup_2026-08-04T19-17-27-498/board.kicad_sch (KiCad schematic)
At the start: 49 parts, among them J11 JST-XH-B6B, J12 USB_C_Receptacle_USB2, J13 JST-XH-B6B, J14 JST-XH-B6B, J4 XT30PW-M, Q19 IRF4905, U4 AP2112K-3.3TRG1(MS), U5 TPS54302, U6 USBLC6-2SC6, U7 ICM-42670-P

Commit message: wip
Parts:
- J11: value JST-XH-B6B -> Enc1
- J12: value USB_C_Receptacle_USB2 -> USB_C_Receptacle_USB2.0_14P
- J13: value JST-XH-B6B -> Enc2; MPN ASDF -> (none)
- J14: value JST-XH-B6B -> Enc3
- TP18, TP19, TP20: MPN 5019 -> (none); Manufacturer Keystone -> (none)
- U4: MPN AP2112K-3.3TRG1(MS) -> (none)
- U5: MPN TPS54302 -> (none); Manufacturer TI -> (none)
- U6: MPN USBLC6-2SC6 -> (none); Manufacturer STMicroelectronics -> (none)
Other:
- moved on the sheet: C45, R40
