File: kicad/stm32_g4_main_board/board/_restore_backup_2026-08-04T19-17-27-498/controller.kicad_sch (KiCad schematic)
At the start: 42 parts, among them IC1 STM32G474MET6TR, J10 STDC, SW1 BOOT, SW2 RESET, Y1 SG-210STF_16.0000ML0

Commit message: wip
Parts:
- added R33: 10k, Resistor_SMD:R_0805_2012Metric, symbol Device:R
- J10: value STDC -> JTAG; footprint Connector_PinHeader_1.27mm:PinHeader_2x07_P1.27mm_Vertical_SMD -> Connector_PinSocket_1.27mm:PinSocket_2x05_P1.27mm_Vertical_SMD; symbol Connector:Conn_ST_STDC14 -> Connector:Conn_ARM_JTAG_SWD_10
- TP10, TP11, TP12, TP13, TP14, TP15, TP16, TP17, TP2, TP21, TP22, TP3, TP4, TP5, TP6, TP7, TP8, TP9: MPN 5019 -> (none); Manufacturer Keystone -> (none)
- Y1: Manufacturer Epson -> (none)
Connections:
- net +3V3: now also J10.1 (VTref), R33.1; no longer J10.3 (VCC)
- net GND: now also J10.3 (GND), J10.9 (GNDDetect); no longer J10.11 (GNDDetect), J10.7 (GND)
- net SWCLK: now also J10.4 (SWCLK/TCK); no longer J10.6 (JCLK/SWCLK)
- net SWDIO: now also J10.2 (SWDIO/TMS); no longer J10.4 (JTMS/SWDIO)
- net SWO: now also J10.6 (SWO/TDO); no longer J10.8 (JTDO/SWO)
- net ~{RESET}: now also J10.10 (~{RESET}), R33.2; no longer J10.12 (~{RST})
- net USART1_RX: no longer names the net of IC1.23 (NC)
- net USART1_RX: no longer J10.13 (VCP_RX)
- net USART1_TX: no longer names the net of IC1.57 (NC)
- net USART1_TX: no longer J10.14 (VCP_TX)
- no-connect marks 6 -> 5
Other:
- note added: "JTAG Header"
- note removed: "STDC/JTAG Header"
