File: kicad/stm32_g4_main_board/board/_restore_backup_2026-08-04T19-17-27-498/motor_channel.kicad_sch (KiCad schematic)
At the start: 14 parts, among them J1 MR30PW-M, U1 DRV8304HRHAR

Commit message: wip
Parts:
- C5: MPN (none) -> NFM21CC223R1H3D
- J1: footprint jaguilar:PinHeader_01x03_Molex_6.35mm -> jaguilar:MR30PWM
Changed lines of the file:
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@@
 					(reference "U1")
 					(unit 1)
-					(variant
-						(name "CountingCurrentParts")
-					)
 				)
 				(path "/be33a253-a895-4341-ac4c-f55475734dc2/5c903e03-aea7-41ae-86fb-f44fc0c1cdbb"
 					(reference "U2")
 					(unit 1)
-					(variant
-						(name "CountingCurrentParts")
-					)
 				)
 				(path "/be33a253-a895-4341-ac4c-f55475734dc2/7222f6b0-274c-4715-84c9-323480ec97a9"
 					(reference "U3")
 					(unit 1)
-					(variant
-						(name "CountingCurrentParts")
-					)
 				)
 			)
@@
 			)
 		)
-		(property "MPN" ""
+		(property "MPN" "NFM21CC223R1H3D"
 			(at 179.07 66.04 0)
 			(hide yes)
@@
 					(reference "C5")
 					(unit 1)
-					(variant
-						(name "CountingCurrentParts")
-					)
 				)
 				(path "/be33a253-a895-4341-ac4c-f55475734dc2/5c903e03-aea7-41ae-86fb-f44fc0c1cdbb"
 					(reference "C17")
 					(unit 1)
-					(variant
-						(name "CountingCurrentParts")
-					)
 				)
 				(path "/be33a253-a895-4341-ac4c-f55475734dc2/7222f6b0-274c-4715-84c9-323480ec97a9"
 					(reference "C29")
 					(unit 1)
-					(variant
-						(name "CountingCurrentParts")
-					)
 				)
 			)
@@
 					(reference "NT1")
 					(unit 1)
-					(variant
-						(name "CountingCurrentParts")
-					)
 				)
 				(path "/be33a253-a895-4341-ac4c-f55475734dc2/5c903e03-aea7-41ae-86fb-f44fc0c1cdbb"
 					(reference "NT2")
 					(unit 1)
-					(variant
-						(name "CountingCurrentParts")
-					)
 				)
 				(path "/be33a253-a895-4341-ac4c-f55475734dc2/7222f6b0-274c-4715-84c9-323480ec97a9"
 					(reference "NT3")
 					(unit 1)
-					(variant
-						(name "CountingCurrentParts")
-					)
 				)
 			)
@@
 					(reference "R3")
 					(unit 1)
-					(variant
-						(name "CountingCurrentParts")
-					)
 				)
 				(path "/be33a253-a895-4341-ac4c-f55475734dc2/5c903e03-aea7-41ae-86fb-f44fc0c1cdbb"
 					(reference "R10")
 					(unit 1)
-					(variant
-						(name "CountingCurrentParts")
-					)
 				)
 				(path "/be33a253-a895-4341-ac4c-f55475734dc2/7222f6b0-274c-4715-84c9-323480ec97a9"
 					(reference "R17")
 					(unit 1)
-					(variant
-						(name "CountingCurrentParts")
-					)
 				)
 			)
@@
 					(reference "C4")
 					(unit 1)
-					(variant
-						(name "CountingCurrentParts")
-					)
 				)
 				(path "/be33a253-a895-4341-ac4c-f55475734dc2/5c903e03-aea7-41ae-86fb-f44fc0c1cdbb"
 					(reference "C16")
 					(unit 1)
-					(variant
-						(name "CountingCurrentParts")
-					)
 				)
 				(path "/be33a253-a895-4341-ac4c-f55475734dc2/7222f6b0-274c-4715-84c9-323480ec97a9"
 					(reference "C28")
 					(unit 1)
-					(variant
-						(name "CountingCurrentParts")
-					)
 				)
 			)
@@
 					(reference "R4")
 					(unit 1)
-					(variant
-						(name "CountingCurrentParts")
-					)
 				)
 				(path "/be33a253-a895-4341-ac4c-f55475734dc2/5c903e03-aea7-41ae-86fb-f44fc0c1cdbb"
 					(reference "R11")
 					(unit 1)
-					(variant
-						(name "CountingCurrentParts")
-					)
 				)
 				(path "/be33a253-a895-4341-ac4c-f55475734dc2/7222f6b0-274c-4715-84c9-323480ec97a9"
 					(reference "R18")
 					(unit 1)
-					(variant
-						(name "CountingCurrentParts")
-					)
 				)
 			)
@@
 					(reference "C2")
 					(unit 1)
-					(variant
-						(name "CountingCurrentParts")
-					)
 				)
 				(path "/be33a253-a895-4341-ac4c-f55475734dc2/5c903e03-aea7-41ae-86fb-f44fc0c1cdbb"
 					(reference "C14")
 					(unit 1)
-					(variant
-						(name "CountingCurrentParts")
-					)
 				)
 				(path "/be33a253-a895-4341-ac4c-f55475734dc2/7222f6b0-274c-4715-84c9-323480ec97a9"
 					(reference "C26")
 					(unit 1)
-					(variant
-						(name "CountingCurrentParts")
-					)
 				)
 			)
@@
 			)
 		)
-		(property "Footprint" "jaguilar:PinHeader_01x03_Molex_6.35mm"
+		(property "Footprint" "jaguilar:MR30PWM"
 			(at 269.24 0.33 0)
 			(hide yes)
@@
 					(reference "J1")
 					(unit 1)
-					(variant
-						(name "CountingCurrentParts")
-					)
 				)
 				(path "/be33a253-a895-4341-ac4c-f55475734dc2/5c903e03-aea7-41ae-86fb-f44fc0c1cdbb"
 					(reference "J2")
 					(unit 1)
-					(variant
-						(name "CountingCurrentParts")
-					)
 				)
 				(path "/be33a253-a895-4341-ac4c-f55475734dc2/7222f6b0-274c-4715-84c9-323480ec97a9"
 					(reference "J3")
 					(unit 1)
-					(variant
-						(name "CountingCurrentParts")
-					)
 				)
 			)
@@
 					(reference "C50")
 					(unit 1)
-					(variant
-						(name "CountingCurrentParts")
-					)
 				)
 				(path "/be33a253-a895-4341-ac4c-f55475734dc2/5c903e03-aea7-41ae-86fb-f44fc0c1cdbb"
 					(reference "C51")
 					(unit 1)
-					(variant
-						(name "CountingCurrentParts")
-					)
 				)
 				(path "/be33a253-a895-4341-ac4c-f55475734dc2/7222f6b0-274c-4715-84c9-323480ec97a9"
 					(reference "C52")
 					(unit 1)
-					(variant
-						(name "CountingCurrentParts")
-					)
 				)
 			)
@@
 					(reference "R1")
 					(unit 1)
-					(variant
-						(name "CountingCurrentParts")
-					)
 				)
 				(path "/be33a253-a895-4341-ac4c-f55475734dc2/5c903e03-aea7-41ae-86fb-f44fc0c1cdbb"
 					(reference "R8")
 					(unit 1)
-					(variant
-						(name "CountingCurrentParts")
-					)
 				)
 				(path "/be33a253-a895-4341-ac4c-f55475734dc2/7222f6b0-274c-4715-84c9-323480ec97a9"
 					(reference "R15")
 					(unit 1)
-					(variant
-						(name "CountingCurrentParts")
-					)
 				)
 			)
@@
 					(reference "R2")
 					(unit 1)
-					(variant
-						(name "CountingCurrentParts")
-					)
 				)
 				(path "/be33a253-a895-4341-ac4c-f55475734dc2/5c903e03-aea7-41ae-86fb-f44fc0c1cdbb"
 					(reference "R9")
 					(unit 1)
-					(variant
-						(name "CountingCurrentParts")
-					)
 				)
 				(path "/be33a253-a895-4341-ac4c-f55475734dc2/7222f6b0-274c-4715-84c9-323480ec97a9"
 					(reference "R16")
 					(unit 1)
-					(variant
-						(name "CountingCurrentParts")
-					)
 				)
 			)
@@
 					(reference "R37")
 					(unit 1)
-					(variant
-						(name "CountingCurrentParts")
-					)
 				)
 				(path "/be33a253-a895-4341-ac4c-f55475734dc2/5c903e03-aea7-41ae-86fb-f44fc0c1cdbb"
 					(reference "R38")
 					(unit 1)
-					(variant
-						(name "CountingCurrentParts")
-					)
 				)
 				(path "/be33a253-a895-4341-ac4c-f55475734dc2/7222f6b0-274c-4715-84c9-323480ec97a9"
 					(reference "R39")
 					(unit 1)
-					(variant
-						(name "CountingCurrentParts")
-					)
 				)
 			)
@@
 					(reference "C3")
 					(unit 1)
-					(variant
-						(name "CountingCurrentParts")
-					)
 				)
 				(path "/be33a253-a895-4341-ac4c-f55475734dc2/5c903e03-aea7-41ae-86fb-f44fc0c1cdbb"
 					(reference "C15")
 					(unit 1)
-					(variant
-						(name "CountingCurrentParts")
-					)
 				)
 				(path "/be33a253-a895-4341-ac4c-f55475734dc2/7222f6b0-274c-4715-84c9-323480ec97a9"
 					(reference "C27")
 					(unit 1)
-					(variant
-						(name "CountingCurrentParts")
-					)
 				)
 			)
@@
 					(reference "C1")
 					(unit 1)
-					(variant
-						(name "CountingCurrentParts")
-					)
 				)
 				(path "/be33a253-a895-4341-ac4c-f55475734dc2/5c903e03-aea7-41ae-86fb-f44fc0c1cdbb"
 					(reference "C13")
 					(unit 1)
-					(variant
-						(name "CountingCurrentParts")
-					)
 				)
 				(path "/be33a253-a895-4341-ac4c-f55475734dc2/7222f6b0-274c-4715-84c9-323480ec97a9"
 					(reference "C25")
 					(unit 1)
-					(variant
-						(name "CountingCurrentParts")
-					)
-				)
-			)
+				)
+			)
