File: kicad/stm32_g4_main_board/board/board.kicad_sch (KiCad schematic)
At the start: 0 parts

Commit message: V1 Board.
Parts:
- added C36: 10u, Capacitor_SMD:C_0805_2012Metric, symbol Device:C
- added C37, C38, C43: 100n, Capacitor_SMD:C_0805_2012Metric, symbol Device:C
- added C39, C40: 22u, Capacitor_SMD:C_0805_2012Metric, symbol Device:C
- added C41: 75p, Capacitor_SMD:C_0805_2012Metric, symbol Device:C
- added C44, C45: 1u, Capacitor_SMD:C_0805_2012Metric, symbol Device:C
- added C46: 2u2, Capacitor_SMD:C_0805_2012Metric, symbol Device:C
- added C47: 10n, Capacitor_SMD:C_0805_2012Metric, symbol Device:C
- added C53, C54, C55, C56: 150u, Capacitor_SMD:CP_Elec_10x10.5, symbol Device:C_Polarized
- added C57: 68n, Capacitor_SMD:C_0805_2012Metric, symbol Device:C
- added D1, D2: SS14, Diode_SMD:D_SMA, symbol Diode:SS14
- added D7: 15V 0.5W, Diode_SMD:D_SOD-123, symbol Device:D_Zener
- added F1: Fuse, jaguilar:Fuse_Blade_XF_507P, symbol Device:Fuse
- added H1, H2, H3, H4: MountingHole, MountingHole:MountingHole_2.2mm_M2, symbol Mechanical:MountingHole
- added J11, J13, J14: JST-XH-B6B, Connector_JST:JST_XH_B6B-XH-A_1x06_P2.50mm_Vertical, symbol Connector:Conn_01x06_Pin
- added J12: USB_C_Receptacle_USB2, jaguilar:C165948_USB-C_SMD-TYPE-C-31-M-12_1, symbol Connector:USB_C_Receptacle_USB2.0_14P
- added J4: XT30PW-M, jaguilar:XT30PWM, symbol jaguilar:XT30PW-M
- added L1: 10u, Inductor_SMD:L_Taiyo-Yuden_NR-60xx, symbol Device:L
- added Q19: IRF4905, Package_TO_SOT_THT:TO-220-3_Vertical, symbol Transistor_FET:IRF4905
- added R26: 511k, Resistor_SMD:R_0805_2012Metric, symbol Device:R
- added R27: 105k, Resistor_SMD:R_0805_2012Metric, symbol Device:R
- added R29, R35: 100k, Resistor_SMD:R_0805_2012Metric, symbol Device:R
- added R30: 13k3, Resistor_SMD:R_0805_2012Metric, symbol Device:R
- added R31, R32: 5k1, Resistor_SMD:R_0805_2012Metric, symbol Device:R
- added R34, R41: 4k7, Resistor_SMD:R_0805_2012Metric, symbol Device:R
- added R36: 150k, Resistor_SMD:R_0805_2012Metric, symbol Device:R
- added R40: 0, Resistor_SMD:R_0805_2012Metric, symbol Device:R
- added TP18: +5V, TestPoint:TestPoint_Keystone_5019_Miniature, symbol Connector:TestPoint
- added TP19: +3V3, TestPoint:TestPoint_Keystone_5019_Miniature, symbol Connector:TestPoint
- added TP20: GND, TestPoint:TestPoint_Keystone_5019_Miniature, symbol Connector:TestPoint
- added U4: AP2112K-3.3TRG1(MS), jaguilar:C22365427_SOT-23-5_L2_9-W1_6-P0_95-LS2_7-BR, symbol lcsc_imported:AP2112K-3_3TRG1(MS)
- added U5: TPS54302, Package_TO_SOT_SMD:SOT-23-6, symbol Regulator_Switching:TPS54302
- added U6: USBLC6-2SC6, Package_TO_SOT_SMD:SOT-23-6, symbol Power_Protection:USBLC6-2SC6
- added U7: ICM-42670-P, Package_LGA:LGA-14_3x2.5mm_P0.5mm_LayoutBorder3x4y, symbol jaguilar:ICM-42670-P
Connections:
- new net: F1.1, J4.1 (+)
- new net: J12.A5 (CC1), R32.1
- new net: J12.B5 (CC2), R31.1
- new net: C57.1, D7.1 (K), F1.2, Q19.3 (S), R35.1, R40.1
- new net: C57.2, D7.2 (A), Q19.1 (G), R35.2, R36.1
- new net: C41.1, R29.2, R30.1, U5.4 (FB)
- new net: R26.2, R27.1, U5.5 (EN)
- new net: C38.2, L1.1, U5.2 (SW)
- new net: C38.1, U5.6 (BOOT)
- new net +3V3: C43.1, C44.2, C46.1, C47.1, J11.6 (Pin_6), J13.6 (Pin_6), J14.6 (Pin_6), R34.1, R41.1, TP19.1, U4.5 (VOUT), U7.5 (VDDIO), U7.8 (VDD)
- new net +5V: C45.2, D1.1 (K), D2.1 (K), TP18.1, U4.1 (VIN), U4.3 (EN)
- new net +BATT: C36.1, C37.1, C53.1, C54.1, C55.1, C56.1, Q19.2 (D), R26.1, R40.2, U5.3 (VIN)
- new net 5V_REG: C39.2, C40.2, C41.2, D1.2 (A), L1.2, R29.1
- new net Controller/USB_D+: U6.6 (I/O1)
- new net Controller/USB_D-: U6.4 (I/O2)
- new net GND: C36.2, C37.2, C39.1, C40.1, C43.2, C44.1, C45.1, C46.2, C47.2, C53.2, C54.2, C55.2, C56.2, J11.2 (Pin_2), J12.SH (SHIELD), J12.[A1,A12,B1,B12] (GND), J13.2 (Pin_2), J14.2 (Pin_2), J4.2 (-), R27.2, R30.2, R31.2, R32.2, R36.2, TP20.1, U4.2 (GND), U5.1 (GND), U6.2 (GND), U7.6 (GND)
- new net I2C1.SCL: R41.2, U7.13 (SCL/SCLK)
- new net I2C1.SDA: R34.2, U7.14 (SDA/SDIO/SDI)
- new net IMU_INT: U7.4 (INT1/INT)
- new net SPI1.MISO: J11.4 (Pin_4), J13.4 (Pin_4), J14.4 (Pin_4)
- new net SPI1.MOSI: J11.5 (Pin_5), J13.5 (Pin_5), J14.5 (Pin_5)
- new net SPI1.SCLK: J11.1 (Pin_1), J13.1 (Pin_1), J14.1 (Pin_1)
- new net USB_D+: J12.A6 (D+), J12.B6 (D+), U6.1 (I/O1)
- new net USB_D-: J12.A7 (D-), J12.B7 (D-), U6.3 (I/O2)
- new net USB_VBUS: D2.2 (A), J12.[A4,A9,B4,B9] (VBUS), U6.5 (VBUS)
- new net ~{ENC1_CS}: J11.3 (Pin_3)
- new net ~{ENC2_CS}: J13.3 (Pin_3)
- new net ~{ENC3_CS}: J14.3 (Pin_3)
- no-connect marks 0 -> 5
Other:
- sheet Motor Channel renamed mchan1
- sheet Motor Channel1 renamed mchan2
- sheet Motor Channel2 renamed mchan3
- sheet Controller ports: added I2C1{SDA SCL}, IMU_INT, SPI1{SCLK MISO MOSI}, USB_D+, USB_D-, {MCOM}, ~{ENC1_CS}, ~{ENC2_CS}, ~{ENC3_CS}; removed none
- sheet mchan1 ports: added {MCOM}; removed none
- sheet mchan2 ports: added {MCOM}; removed none
- sheet mchan3 ports: added {MCOM}; removed none
- note added: "3V3 Regulator"
- note added: "5V Regulator"
- note added: "Accelerometer/Gyroscope"
- note added: "Bulk Capacitance"
- note added: "Bypass caps for VDD (C43 & C46) and VDDIO (C47)"
- note added: "Encoder headers"
- note added: "Plug & Anti-Spark"
- note added: "Prevents spark by gradually enabling p-fet during the charge time of C_{gs}, approx 34ms (5 * tau, tau = 6.8ms)."
- note added: "USB Receptacle"

Commit message: WIP - v2 board
Parts:
- removed H3: MountingHole, MountingHole:MountingHole_2.2mm_M2, symbol Mechanical:MountingHole
- D7: value 15V 0.5W -> 10V 0.5W
- H1, H2, H4: footprint MountingHole:MountingHole_2.2mm_M2 -> MountingHole:MountingHole_2.2mm_M2_Pad_Via; symbol Mechanical:MountingHole -> Mechanical:MountingHole_Pad
- R40: footprint Resistor_SMD:R_0805_2012Metric -> Resistor_SMD:R_1206_3216Metric
Connections:
- net GND: now also H1.1, H2.1, H4.1
Other:
- sheet Controller ports: added SPI1{SPI}; removed SPI1{SCLK MISO MOSI}
- sheet mchan1 ports: added {SPI}; removed none
- sheet mchan2 ports: added {SPI}; removed none
- sheet mchan3 ports: added {SPI}; removed none
- moved on the sheet: J11, J13, J14, U6
