File: kicad/stm32_g4_main_board/board/controller.kicad_sch (KiCad schematic)
At the start: 0 parts

Commit message: V1 Board.
Parts:
- added C10, C12, C18, C20, C48, C6, C8: 100n, Capacitor_SMD:C_0603_1608Metric, symbol Device:C
- added C22: 1u, Capacitor_SMD:C_0603_1608Metric, symbol Device:C
- added C32, C34, C49: 100n, Capacitor_SMD:C_0805_2012Metric, symbol Device:C
- added D3, D4, D5, D6: WS2812B, LED_SMD:LED_WS2812B_PLCC4_5.0x5.0mm_P3.2mm, symbol LED:WS2812B
- added IC1: STM32G474MET6TR, Package_QFP:LQFP-80_12x12mm_P0.5mm, symbol STM32G474MET6TR:STM32G474MET6TR
- added J10: STDC, Connector_PinHeader_1.27mm:PinHeader_2x07_P1.27mm_Vertical_SMD, symbol Connector:Conn_ST_STDC14
- added R22, R24, R25: 10k, Resistor_SMD:R_0805_2012Metric, symbol Device:R
- added R23: 82k, Resistor_SMD:R_0805_2012Metric, symbol Device:R
- added SW1: BOOT, Button_Switch_THT:SW_PUSH_6mm_H5mm, symbol Switch:SW_Push
- added SW2: RESET, Button_Switch_THT:SW_PUSH_6mm_H5mm, symbol Switch:SW_Push
- added TP10: INHA, TestPoint:TestPoint_Keystone_5019_Miniature, symbol Connector:TestPoint
- added TP11: INHB, TestPoint:TestPoint_Keystone_5019_Miniature, symbol Connector:TestPoint
- added TP12: INHC, TestPoint:TestPoint_Keystone_5019_Miniature, symbol Connector:TestPoint
- added TP13: INL, TestPoint:TestPoint_Keystone_5019_Miniature, symbol Connector:TestPoint
- added TP14: SOA, TestPoint:TestPoint_Keystone_5019_Miniature, symbol Connector:TestPoint
- added TP15: SOB, TestPoint:TestPoint_Keystone_5019_Miniature, symbol Connector:TestPoint
- added TP16: SOC, TestPoint:TestPoint_Keystone_5019_Miniature, symbol Connector:TestPoint
- added TP17: CAL, TestPoint:TestPoint_Keystone_5019_Miniature, symbol Connector:TestPoint
- added TP2: SCLK, TestPoint:TestPoint_Keystone_5019_Miniature, symbol Connector:TestPoint
- added TP21: IMU_INT, TestPoint:TestPoint_Keystone_5019_Miniature, symbol Connector:TestPoint
- added TP22: VBATT_SENSE, TestPoint:TestPoint_Keystone_5019_Miniature, symbol Connector:TestPoint
- added TP3: MISO, TestPoint:TestPoint_Keystone_5019_Miniature, symbol Connector:TestPoint
- added TP4: MOSI, TestPoint:TestPoint_Keystone_5019_Miniature, symbol Connector:TestPoint
- added TP5: CS, TestPoint:TestPoint_Keystone_5019_Miniature, symbol Connector:TestPoint
- added TP6: SDA, TestPoint:TestPoint_Keystone_5019_Miniature, symbol Connector:TestPoint
- added TP7: SCL, TestPoint:TestPoint_Keystone_5019_Miniature, symbol Connector:TestPoint
- added TP8: EN, TestPoint:TestPoint_Keystone_5019_Miniature, symbol Connector:TestPoint
- added TP9: ~{FAULT}, TestPoint:TestPoint_Keystone_5019_Miniature, symbol Connector:TestPoint
- added Y1: SG-210STF_16.0000ML0, jaguilar:SG-210STF_EPS, symbol SG-210STF_16_0000ML0:SG-210STF_16.0000ML0
Connections:
- net M1.INHA: now also IC1.56 (M1_PHASEA_OUT), TP10.1
- new net: D3.2 (DOUT), D4.4 (DIN)
- new net: R25.2, Y1.1 (~{ST})
- new net: D5.2 (DOUT), D6.4 (DIN)
- new net: D4.2 (DOUT), D5.4 (DIN)
- new net +3V3: C10.1, C12.1, C18.1, C20.1, C22.1, C34.1, C48.1, C6.1, C8.1, D3.1 (VDD), D4.1 (VDD), D5.1 (VDD), D6.1 (VDD), IC1.1 (VBAT), IC1.28 (VREF+), IC1.29 (VDDA), IC1.[16,41,51,62,80] (VDD), J10.3 (VCC), R25.1, SW1.2, Y1.4 (VCC)
- new net +BATT: R23.1
- new net BOOT0: IC1.77 (BOOT0), R22.1, SW1.1
- new net BYPASS_CLOCK: IC1.5 (PF0-OSC_IN), Y1.3 (OUT)
- new net CAL: IC1.25 (MOTOR_CAL), TP17.1
- new net EN: IC1.24 (MOTOR_EN), TP8.1
- new net GND: C10.2, C12.2, C18.2, C20.2, C22.2, C32.2, C34.2, C48.2, C49.2, C6.2, C8.2, D3.3 (VSS), D4.3 (VSS), D5.3 (VSS), D6.3 (VSS), IC1.27 (VSSA), IC1.[15,40,50,61,79] (VSS), J10.11 (GNDDetect), J10.5 (GND), J10.7 (GND), R22.2, R24.2, SW2.1, Y1.2 (_GND)
- new net I2C1.SCL: IC1.65 (IMU_SCL), TP7.1
- new net I2C1.SDA: IC1.76 (IMU_SDA), TP6.1
- new net IMU_INT: IC1.42 (IMU_INT), TP21.1
- new net LED_DATA: D3.4 (DIN), IC1.75 (LED_DATA)
- new net M1.INHB: IC1.9 (M1_PHASEB_OUT), TP11.1
- new net M1.INHC: IC1.58 (M1_PHASEC_OUT), TP12.1
- new net M1.INL: IC1.49 (~{M1_COAST}), TP13.1
- new net M1.SOA: IC1.32 (M1_PHASEC_SENSE), TP14.1
- new net M1.SOB: IC1.12 (M1_PHASEA_SENSE), TP15.1
- new net M1.SOC: IC1.13 (M1_PHASEB_SENSE), TP16.1
- new net M1.~{FAULT}: IC1.31 (~{M1_FAULT}), TP9.1
- new net M2.INHA: IC1.52 (M2_PHASEA_OUT)
- new net M2.INHB: IC1.53 (M2_PHASEB_OUT)
- new net M2.INHC: IC1.78 (M2_PHASEC_OUT)
- new net M2.INL: IC1.48 (~{M2_COAST})
- new net M2.SOA: IC1.45 (M2_PHASEA_SENSE)
- new net M2.SOB: IC1.21 (M2_PHASEB_SENSE)
- new net M2.SOC: IC1.36 (M2_PHASEC_SENSE)
- new net M2.~{FAULT}: IC1.46 (~{M2_FAULT})
- new net M3.INHA: IC1.26 (M3_PHASEA_OUT)
- new net M3.INHB: IC1.10 (M3_PHASEB_OUT)
- new net M3.INHC: IC1.54 (M3_PHASEC_OUT)
- new net M3.INL: IC1.47 (~{M3_COAST})
- new net M3.SOA: IC1.8 (M3_PHASEA_SENSE)
- new net M3.SOB: IC1.30 (M3_PHASEC_SENSE)
- new net M3.SOC: IC1.22 (M3_PHASEB_SENSE)
- new net M3.~{FAULT}: IC1.44 (~{M3_FAULT})
- new net SPI1.MISO: IC1.20 (ENC_MISO), TP3.1
- new net SPI1.MOSI: IC1.74 (ENC_MOSI), TP4.1
- new net SPI1.SCLK: IC1.19 (ENC_SCLK), TP2.1
- new net SWCLK: IC1.64 (SYS_JTCK-SWCLK), J10.6 (JCLK/SWCLK)
- new net SWDIO: IC1.63 (SYS_JTMS-SWDIO), J10.4 (JTMS/SWDIO)
- new net SWO: IC1.72 (SYS_JTDO-SWO), J10.8 (JTDO/SWO)
- new net USART1_RX: IC1.23 (USART1_RX), J10.13 (VCP_RX)
- new net USART1_TX: IC1.57 (USART1_TX), J10.14 (VCP_TX)
- new net USB_D+: IC1.60 (USB_D+)
- new net USB_D-: IC1.59 (USB_D-)
- new net VBATT_SENSE: C32.1, IC1.37 (VBATT_SENSE), R23.2, R24.1, TP22.1
- new net ~{ENC1_CS}: IC1.73 (~{ENC1_CS}), TP5.1
- new net ~{ENC2_CS}: IC1.18 (~{ENC2_CS})
- new net ~{ENC3_CS}: IC1.55 (~{ENC3_CS})
- new net ~{RESET}: C49.1, IC1.7 (PG10-NRST), J10.12 (~{RST}), SW2.2
- no-connect marks 0 -> 6
Other:
- note added: "Analog decoupling"
- note added: "Battery level sensing"
- note added: "Boot button"
- note added: "Digital decoupling"
- note added: "External Bypass Clock"
- note added: "LED Array"
- note added: "Note: one cap for VBAT<->GND"
- note added: "Note: one of these pairs should be placed at vref+."
- note added: "Reset button"
- note added: "STDC/JTAG Header"

Commit message: WIP - v2 board
Parts:
- removed C10, C12, C18, C20, C48, C6, C8: 100n, Capacitor_SMD:C_0603_1608Metric, symbol Device:C
- removed C22: 1u, Capacitor_SMD:C_0603_1608Metric, symbol Device:C
- removed IC1: STM32G474MET6TR, Package_QFP:LQFP-80_12x12mm_P0.5mm, symbol STM32G474MET6TR:STM32G474MET6TR
- removed TP5: CS, TestPoint:TestPoint_Keystone_5019_Miniature, symbol Connector:TestPoint
- added C24, C42, C58, C59, C60, C61, C62: 100n, Capacitor_SMD:C_0603_1608Metric, symbol Device:C
- added C30: 1u, Capacitor_SMD:C_0603_1608Metric, symbol Device:C
- added U17: STM32G474METx, Package_QFP:LQFP-80_12x12mm_P0.5mm, symbol MCU_ST_STM32G4:STM32G474METx
- J10: footprint Connector_PinHeader_1.27mm:PinHeader_2x07_P1.27mm_Vertical_SMD -> jaguilar:FTSH-107-01-L-DV-K-A; MPN FTSH-105-01-L-DV-K -> FTSH-107-01-L-DV-K-A
- TP22: value VBATT_SENSE -> VBS
Connections:
- net +3V3: now also C24.1, C30.1, C42.1, C58.1, C59.1, C60.1, C61.1, C62.1, U17.1 (VBAT), U17.16 (VDD), U17.28 (VREF+), U17.29 (VDDA), U17.41 (VDD), U17.51 (VDD), U17.62 (VDD), U17.80 (VDD)
- net BOOT0: now also U17.77 (PB8)
- net BYPASS_CLOCK: now also U17.5 (PF0)
- net CAL: now also U17.3 (PC14)
- net EN: now also U17.2 (PC13)
- net GND: now also C24.2, C30.2, C42.2, C58.2, C59.2, C60.2, C61.2, C62.2, U17.15 (VSS), U17.27 (VSSA), U17.40 (VSS), U17.50 (VSS), U17.61 (VSS), U17.79 (VSS)
- net I2C1.SCL: now also U17.65 (PA15)
- net I2C1.SDA: now also U17.76 (PB7)
- net IMU_INT: now also U17.38 (PE15)
- net LED_DATA: now also U17.75 (PB6)
- net M1.INHA: now also U17.56 (PA8)
- net M1.INHB: now also U17.34 (PE11)
- net M1.INHC: now also U17.58 (PA10)
- net M1.INL: now also U17.49 (PD10)
- net M1.SOA: now also U17.24 (PB0)
- net M1.SOB: now also U17.21 (PA7)
- net M1.SOC: now also U17.32 (PE9)
- net M1.~{FAULT}: now also U17.25 (PB1)
- net M2.INHA: now also U17.52 (PC6)
- net M2.INHB: now also U17.53 (PC7)
- net M2.INHC: now also U17.78 (PB9)
- net M2.INL: now also U17.48 (PD9)
- net M2.SOA: now also U17.45 (PB14)
- net M2.SOB: now also U17.22 (PC4)
- net M2.SOC: now also U17.36 (PE13)
- net M2.~{FAULT}: now also U17.31 (PE8)
- net M3.INHA: now also U17.26 (PB2)
- net M3.INHB: now also U17.10 (PC2)
- net M3.INHC: now also U17.54 (PC8)
- net M3.INL: now also U17.47 (PD8)
- net M3.SOA: now also U17.43 (PB12)
- net M3.SOB: now also U17.46 (PB15)
- net M3.SOC: now also U17.30 (PE7)
- net M3.~{FAULT}: now also U17.35 (PE12)
- net SPI1.MISO: now also U17.20 (PA6)
- net SPI1.MOSI: now also U17.74 (PB5)
- net SPI1.SCLK: now also U17.19 (PA5)
- net SWCLK: now also U17.64 (PA14)
- net SWDIO: now also U17.63 (PA13)
- net SWO: now also U17.72 (PB3)
- net USART1_RX: now also U17.23 (PC5)
- net USART1_TX: now also U17.57 (PA9)
- net USB_D+: now also U17.60 (PA12)
- net USB_D-: now also U17.59 (PA11)
- net VBATT_SENSE: now also U17.37 (PE14)
- net ~{ENC1_CS}: now also U17.73 (PB4)
- net ~{ENC2_CS}: now also U17.18 (PA4)
- net ~{ENC3_CS}: now also U17.55 (PC9)
- net ~{RESET}: now also U17.7 (PG10)
- new net M1.~{COAST}: U17.33 (PE10)
- new net M1.~{CS}: U17.39 (PB10)
- new net M2.~{CS}: U17.42 (PB11)
- new net M3.~{CS}: U17.44 (PB13)
- no-connect marks 6 -> 18
Other:
- note removed: "Analog decoupling"
- note removed: "Digital decoupling"
- note removed: "Note: one cap for VBAT<->GND"
- note removed: "Note: one of these pairs should be placed at vref+."
